Commit message: Adjust origin position for joint6output_to_wand
Updated the z-coordinate of the origin for the joint6output_to_wand joint.

File: ros_sim/resource/robots/mycobot_280_pi/mycobot_280_pi_mod.urdf (robot description, URDF)
Before this commit: robot firefighter, 11 links, 10 joints
Joints:
- joint joint6output_to_wand: origin xyz=-0.028284271 -0.028284271 0.02 rpy=0.0 0.0 0.0 -> xyz=-0.028284271 -0.028284271 0.035 rpy=0.0 0.0 0.0
